File: hardware/7-seg_x_8-digRev2.sch (EAGLE design)
At the start: 25 parts, among them U1 SN74LV164APW

Commit message: Updating to latest versions of PCB files
Parts:
- FRAME1: DATECODE 07OCT2014 -> 13OCT2014
Changed lines of the file:
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@@
 <attribute name="CNAME" value="C.Schnarel"/>
 <attribute name="CREVISION" value="Rev 2"/>
-<attribute name="DATECODE" value="07OCT2014"/>
+<attribute name="DATECODE" value="13OCT2014"/>
 <attribute name="DESIGNER" value="C.Schnarel"/>
 </part>
